File: YaLD_amp.sch (KiCad schematic (older format))
At the start: 48 parts, among them U10 IRF7103, U11 IRF7103, U12 IRF7103, U13 IRF7103, U14 IRF7103, U15 IRF7103, U16 IRF7103, U17 IRF7103, U18 IRF7103, U3 IRF7103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

Commit message: changed outputs to 3.5mm pitch
Parts:
- R10, R11, R12, R13, R14, R15, R16, R17, R18, R19, R20, R21, R22, R23, R24, R25, R26, R27, R28, R29, R30, R31, R32, R33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: symbol R -> R-RESCUE-YaLD
